File: Mqtt32output/Mqtt32output.kicad_pcb (KiCad board)
At the start: 2 copper layers, 97.8 x 81.3 mm, 25 parts, among them J1 OUTPUT 0-7, J2 OUTPUT 8-15, J3 OUTPUT 16-23, J4 OUTPUT 24-31, SW1 DIP SWITCH NODE NUMBER 0..3, U2 74HC595, U4 74HC595, U6 74HC595, U8 74HC595, X1 0V - 5V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

Commit message: Fix component placement, and GND connexion + board size on inputs
Parts:
- removed REF**: MountingHole_2.5mm, MountingHole:MountingHole_2.5mm
- added G***: LOGO, _Extra_footprints:shark, F.Cu at (138.4, 61.0)
- added R8: 10k, Resistor_THT:R_Axial_DIN0207_L6.3mm_D2.5mm_P2.54mm_Vertical, F.Cu at (144.8, 55.9)
Connections:
- A1 pad 1: Net-(A1-Pad1) -> (no net)
- A1 pad 10: Net-(A1-Pad10) -> (no net)
- A1 pad 11: Net-(A1-Pad11) -> (no net)
- A1 pad 12: Net-(A1-Pad12) -> (no net)
- A1 pad 13: Net-(A1-Pad13) -> (no net)
- A1 pad 14: Net-(A1-Pad14) -> (no net)
- A1 pad 15: Net-(A1-Pad15) -> (no net)
- A1 pad 16: Net-(A1-Pad16) -> (no net)
- A1 pad 17: Net-(A1-Pad17) -> (no net)
- A1 pad 18: Net-(A1-Pad18) -> (no net)
- A1 pad 2: Net-(A1-Pad2) -> (no net)
- A1 pad 23: Net-(A1-Pad23) -> (no net)
- A1 pad 24: Net-(A1-Pad24) -> (no net)
- A1 pad 25: Net-(A1-Pad25) -> (no net)
- A1 pad 28: Net-(A1-Pad28) -> (no net)
- A1 pad 3: Net-(A1-Pad3) -> (no net)
- A1 pad 30: Net-(A1-Pad30) -> (no net)
- A1 pad 6: Net-(A1-Pad6) -> (no net)
- A1 pad 7: Net-(A1-Pad7) -> (no net)
- A1 pad 8: Net-(A1-Pad8) -> (no net)
- A1 pad 9: Net-(A1-Pad9) -> (no net)
- U2 pad 13: Earth -> Net-(A1-Pad22)
- U4 pad 13: Earth -> Net-(A1-Pad22)
- U6 pad 13: Earth -> Net-(A1-Pad22)
- U8 pad 13: Earth -> Net-(A1-Pad22)
- U8 pad 9: Net-(U8-Pad9) -> (no net)
Routing:
- net +5V: track 228.3 -> 132.8 mm
- net Earth: track 355.3 -> 265.4 mm
- net Net-(A1-Pad22): track 0.00 -> 83.0 mm
- net +24V: track 188.3 -> 168.2 mm
- net Net-(A1-Pad26): track 55.6 -> 62.2 mm
- net Net-(U2-Pad9): track 61.3 -> 67.1 mm
- net Net-(A1-Pad19): track 74.4 -> 68.8 mm
- net Net-(A1-Pad21): track 98.8 -> 94.2 mm
- net Net-(A1-Pad20): track 100.5 -> 96.1 mm
- net Net-(J3-PadA6): track 16.9 -> 20.7 mm
- net Net-(U4-Pad9): track 7.23 -> 9.49 mm
- net Net-(U2-Pad15): track 13.4 -> 12.5 mm
- net Net-(J3-PadA2): track 16.9 -> 17.7 mm
- net Net-(J2-PadA6): track 12.1 -> 11.4 mm
- net Net-(J2-PadA2): track 12.1 -> 11.4 mm
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Other:
- board text added: "+0V"
- board text added: "32 OUTPUTS V2.1 - MQTT github.com/ antibarbie/io- hardware"
- board text added: "JLCJLCJLCJLC"
- board text added: "Mainly On : OK Mainly Off: Init failed Blink Fast : MQTT error Blink Slow : No CNX Still : Reset needed"
- board text removed: "32 OUTPUTS V2.0 - MQTT github.com/ antibarbie/io- hardware"
